Commit message: [update] add tag(collision, inertial)

File: worlds/open_manipulator.urdf.xacro (robot description, xacro)
@@ -37,10 +37,10 @@
       <material name="grey"/>
     </visual>
-    <!--    <collision>
+    <collision>
       <origin xyz="0 0 0" rpy="0 0 0"/>
       <geometry>
         <mesh filename="package://open_manipulator_ign/models/openmanipulator/meshes/chain_link1.stl" scale="0.001 0.001 0.001"/>
       </geometry>
-    </collision>-->
+    </collision>
     <!--    <inertial>
       <origin xyz="0 0 0" />
@@ -50,5 +50,5 @@
                izz="0.1" />
     </inertial>-->
-    <!--     <inertial>
+    <inertial>
       <origin xyz="3.0876154e-04 0.0000000e+00 -1.2176461e-04" />
       <mass value="7.9119962e-02" />
@@ -56,5 +56,5 @@
                iyy="2.1898364e-05" iyz="0.0"
                izz="1.9267361e-05" />
-    </inertial>-->
+    </inertial>
   </link>
   <!-- Joint 1 -->
@@ -77,10 +77,10 @@
       <material name="grey"/>
     </visual>
-    <!--    <collision>
+    <collision>
       <origin xyz="0 0 0.019" rpy="0 0 0"/>
       <geometry>
         <mesh filename="package://open_manipulator_ign/models/openmanipulator/meshes/chain_link2.stl" scale="0.001 0.001 0.001"/>
       </geometry>
-    </collision>-->
+    </collision>
     <!--    <inertial>
       <origin xyz="0 0 0" />
@@ -90,5 +90,5 @@
                izz="0.1" />
     </inertial>-->
-    <!--     <inertial>
+    <inertial>
       <origin xyz="-3.0184870e-04 5.4043684e-04 ${0.018 + 2.9433464e-02}" />
       <mass value="9.8406837e-02" />
@@ -96,5 +96,5 @@
                iyy="3.2689329e-05" iyz="2.8511935e-08"
                izz="1.8850320e-05" />
-    </inertial>-->
+    </inertial>
   </link>
   <!--  Joint 2 -->
@@ -117,10 +117,10 @@
       <material name="grey"/>
     </visual>
-    <!--    <collision>
+    <collision>
       <origin xyz="0 0 0" rpy="0 0 0"/>
       <geometry>
         <mesh filename="package://open_manipulator_ign/models/openmanipulator/meshes/chain_link3.stl" scale="0.001 0.001 0.001"/>
       </geometry>
-    </collision>-->
+    </collision>
     <!--    <inertial>
       <origin xyz="0 0 0" />
@@ -130,5 +130,5 @@
                izz="0.1" />
     </inertial>-->
-    <!--     <inertial>
+    <inertial>
       <origin xyz="1.0308393e-02 3.7743363e-04 1.0170197e-01" />
       <mass value="1.3850917e-01" />
@@ -136,5 +136,5 @@
                iyy="3.4290447e-04" iyz="-1.5717516e-06"
                izz="6.0346498e-05" />
-    </inertial>-->
+    </inertial>
   </link>
   <!--  Joint 3 -->
@@ -157,10 +157,10 @@
       <material name="grey"/>
     </visual>
-    <!--    <collision>
+    <collision>
       <origin xyz="0 0 0" rpy="0 0 0"/>
       <geometry>
         <mesh filename="package://open_manipulator_ign/models/openmanipulator/meshes/chain_link4.stl" scale="0.001 0.001 0.001"/>
       </geometry>
-    </collision>-->
+    </collision>
     <!--    <inertial>
       <origin xyz="0 0 0" />
@@ -170,5 +170,5 @@
                izz="0.1" />
     </inertial>-->
-    <!--     <inertial>
+    <inertial>
       <origin xyz="9.0909590e-02 3.8929816e-04 2.2413279e-04" />
       <mass value="1.3274562e-01" />
@@ -176,5 +176,5 @@
                iyy="2.4230292e-04" iyz="1.1559550e-08"
                izz="2.5155057e-04" />
-    </inertial>-->
+    </inertial>
   </link>
   <!--  Joint 4 -->
@@ -197,10 +197,10 @@
       <material name="grey"/>
     </visual>
-    <!--    <collision>
+    <collision>
       <origin xyz="0 0 0" rpy="0 0 0"/>
       <geometry>
         <mesh filename="package://open_manipulator_ign/models/openmanipulator/meshes/chain_link5.stl" scale="0.001 0.001 0.001"/>
       </geometry>
-    </collision>-->
+    </collision>
     <!--    <inertial>
       <origin xyz="0 0 0" />
@@ -210,5 +210,5 @@
                izz="0.1" />
     </inertial>-->
-    <!--     <inertial>
+    <inertial>
       <origin xyz="4.4206755e-02 3.6839985e-07 8.9142216e-03" />
       <mass value="1.4327573e-01" />
@@ -216,5 +216,5 @@
                iyy="7.5980465e-05" iyz="0.0"
                izz="9.3127351e-05" />
-    </inertial>-->
+    </inertial>
   </link>
   <!--  Gripper link -->
@@ -227,10 +227,10 @@
       <material name="grey"/>
     </visual>
-    <!--    <collision>
+    <collision>
       <origin xyz="0.0 0.0 0" rpy="0 0 0"/>
       <geometry>
         <mesh filename="package://open_manipulator_ign/models/openmanipulator/meshes/chain_link_grip_l.stl" scale="0.001 0.001 0.001"/>
       </geometry>
-    </collision>-->
+    </collision>
     <!--    <inertial>
       <origin xyz="0 0 0" />
@@ -240,5 +240,5 @@
                izz="1.0e-03" />
     </inertial>-->
-    <!--     <inertial>
+    <inertial>
       <origin xyz="${0.028 + 8.3720668e-03} ${0.0246 + 9.9696160e-03} -4.2836895e-07" />
       <mass value="3.2218127e-02" />
@@ -246,5 +246,5 @@
                iyy="2.2552871e-05" iyz="-3.1463634e-10"
                izz="1.7605306e-05" />
-    </inertial>-->
+    </inertial>
   </link>
   <!--  Gripper joint -->
@@ -267,10 +267,10 @@
       <material name="grey"/>
     </visual>
-    <!--    <collision>
+    <collision>
       <origin xyz="0.0 -0.0 0" rpy="0 0 0"/>
       <geometry>
         <mesh filename="package://open_manipulator_ign/models/openmanipulator/meshes/chain_link_grip_r.stl" scale="0.001 0.001 0.001"/>
       </geometry>
-    </collision>-->
+    </collision>
     <!--    <inertial>
       <origin xyz="0 0 0" />
@@ -280,5 +280,5 @@
                izz="1.0e-03" />
     </inertial>-->
-    <!--     <inertial>
+    <inertial>
       <origin xyz="${0.028 + 8.3720668e-03} ${-0.0246 - 9.9696160e-03} -4.2836895e-07" />
       <mass value="3.2218127e-02" />
@@ -286,5 +286,5 @@
                iyy="2.2552871e-05" iyz="-3.1463634e-10"
                izz="1.7605306e-05" />
-    </inertial>-->
+    </inertial>
   </link>
   <!--  Gripper joint sub -->
@@ -314,9 +314,9 @@
       <material name="red"/>
      </visual>
-    <!--    <inertial>
+    <inertial>
       <origin xyz="0.0 0.0 0.0" rpy="0 0 0"/>
       <mass value="0.001"/>
       <inertia ixx="1.0e-06" ixy="0.0" ixz="0.0" iyy="1.0e-06" iyz="0.0" izz="1.0e-06" />
-    </inertial>-->
+    </inertial>
   </link>
 </robot>
