Commit message: [update] ignitionで表示

File: worlds/openManipulator/open_manipulator.urdf (robot description, URDF)
Before this commit: robot open_manipulator, 9 links, 8 joints
Links:
- link end_effector_link: mass None -> 0.001
- link gripper_link: mass None -> 3.2218127e-02; geometry collision mesh filename=/home/kaito/ign_ws/src/open_manipulator_ign/models/openmani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 scale=0.001 0.001 0.001; visual mesh filename=/home/kaito/ign_ws/src/open_manipulator_ign/models/openmani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 scale=0.001 0.001 0.001
- link gripper_link_sub: mass None -> 3.2218127e-02; geometry collision mesh filename=/home/kaito/ign_ws/src/open_manipulator_ign/models/openmani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 scale=0.001 0.001 0.001; visual mesh filename=/home/kaito/ign_ws/src/open_manipulator_ign/models/openmani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 scale=0.001 0.001 0.001
- link link1: mass None -> 7.9119962e-02; geometry collision mesh filename=/home/kaito/ign_ws/src/open_manipulator_ign/models/openmani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 scale=0.001 0.001 0.001; visual mesh filename=/home/kaito/ign_ws/src/open_manipulator_ign/models/openmani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 scale=0.001 0.001 0.001
- link link2: mass None -> 9.8406837e-02; geometry collision mesh filename=/home/kaito/ign_ws/src/open_manipulator_ign/models/openmani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 scale=0.001 0.001 0.001; visual mesh filename=/home/kaito/ign_ws/src/open_manipulator_ign/models/openmani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 scale=0.001 0.001 0.001
- link link3: mass None -> 1.3850917e-01; geometry collision mesh filename=/home/kaito/ign_ws/src/open_manipulator_ign/models/openmani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 scale=0.001 0.001 0.001; visual mesh filename=/home/kaito/ign_ws/src/open_manipulator_ign/models/openmani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 scale=0.001 0.001 0.001
- link link4: mass None -> 1.3274562e-01; geometry collision mesh filename=/home/kaito/ign_ws/src/open_manipulator_ign/models/openmani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 scale=0.001 0.001 0.001; visual mesh filename=/home/kaito/ign_ws/src/open_manipulator_ign/models/openmani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 scale=0.001 0.001 0.001
- link link5: mass None -> 1.4327573e-01; geometry collision mesh filename=/home/kaito/ign_ws/src/open_manipulator_ign/models/openmani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 scale=0.001 0.001 0.001; visual mesh filename=/home/kaito/ign_ws/src/open_manipulator_ign/models/openmani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 scale=0.001 0.001 0.001

File: worlds/openManipulator/open_manipulator.urdf.xacro (robot description, xacro)
@@ -5,5 +5,5 @@
   <!--  <xacro:include filename="$(find open_manipulator_description)/urdf/open_manipulator.gazebo.xacro" />-->
   <!-- Import Rviz colors -->
-  <xacro:include filename="$(find open_manipulator_ign)/worlds/materials.xacro" />
+  <xacro:include filename="$(find open_manipulator_ign)/worlds/openManipulator/materials.xacro" />
   <!-- Transmission macro -->
   <!--<xacro:macro name="SimpleTransmission" params="joint n">
@@ -33,12 +33,12 @@
       <origin xyz="0 0 0" rpy="0 0 0"/>
       <geometry>
-        <mesh filename="package://open_manipulator_ign/models/openmanipulator/meshes/chain_link1.stl" scale="0.001 0.001 0.001"/>
-      </geometry>
-      <material name="grey"/>
-    </visual>
-    <collision>
-      <origin xyz="0 0 0" rpy="0 0 0"/>
-      <geometry>
-        <mesh filename="package://open_manipulator_ign/models/openmanipulator/meshes/chain_link1.stl" scale="0.001 0.001 0.001"/>
+        <mesh filename="/home/kaito/ign_ws/src/open_manipulator_ign/models/openmanipulator/meshes/chain_link1.stl" scale="0.001 0.001 0.001"/>
+      </geometry>
+      <material name="grey"/>
+    </visual>
+    <collision>
+      <origin xyz="0 0 0" rpy="0 0 0"/>
+      <geometry>
+        <mesh filename="/home/kaito/ign_ws/src/open_manipulator_ign/models/openmanipulator/meshes/chain_link1.stl" scale="0.001 0.001 0.001"/>
       </geometry>
     </collision>
@@ -73,5 +73,5 @@
       <origin xyz="0 0 0.019" rpy="0 0 0"/>
       <geometry>
-        <mesh filename="package://open_manipulator_ign/models/openmanipulator/meshes/chain_link2.stl" scale="0.001 0.001 0.001"/>
+        <mesh filename="/home/kaito/ign_ws/src/open_manipulator_ign/models/openmanipulator/meshes/chain_link2.stl" scale="0.001 0.001 0.001"/>
       </geometry>
       <material name="grey"/>
@@ -80,5 +80,5 @@
       <origin xyz="0 0 0.019" rpy="0 0 0"/>
       <geometry>
-        <mesh filename="package://open_manipulator_ign/models/openmanipulator/meshes/chain_link2.stl" scale="0.001 0.001 0.001"/>
+        <mesh filename="/home/kaito/ign_ws/src/open_manipulator_ign/models/openmanipulator/meshes/chain_link2.stl" scale="0.001 0.001 0.001"/>
       </geometry>
     </collision>
@@ -113,12 +113,12 @@
       <origin xyz="0 0 0" rpy="0 0 0"/>
       <geometry>
-        <mesh filename="package://open_manipulator_ign/models/openmanipulator/meshes/chain_link3.stl" scale="0.001 0.001 0.001"/>
-      </geometry>
-      <material name="grey"/>
-    </visual>
-    <collision>
-      <origin xyz="0 0 0" rpy="0 0 0"/>
-      <geometry>
-        <mesh filename="package://open_manipulator_ign/models/openmanipulator/meshes/chain_link3.stl" scale="0.001 0.001 0.001"/>
+        <mesh filename="/home/kaito/ign_ws/src/open_manipulator_ign/models/openmanipulator/meshes/chain_link3.stl" scale="0.001 0.001 0.001"/>
+      </geometry>
+      <material name="grey"/>
+    </visual>
+    <collision>
+      <origin xyz="0 0 0" rpy="0 0 0"/>
+      <geometry>
+        <mesh filename="/home/kaito/ign_ws/src/open_manipulator_ign/models/openmanipulator/meshes/chain_link3.stl" scale="0.001 0.001 0.001"/>
       </geometry>
     </collision>
@@ -153,12 +153,12 @@
       <origin xyz="0 0 0" rpy="0 0 0"/>
       <geometry>
-        <mesh filename="package://open_manipulator_ign/models/openmanipulator/meshes/chain_link4.stl" scale="0.001 0.001 0.001"/>
-      </geometry>
-      <material name="grey"/>
-    </visual>
-    <collision>
-      <origin xyz="0 0 0" rpy="0 0 0"/>
-      <geometry>
-        <mesh filename="package://open_manipulator_ign/models/openmanipulator/meshes/chain_link4.stl" scale="0.001 0.001 0.001"/>
+        <mesh filename="/home/kaito/ign_ws/src/open_manipulator_ign/models/openmanipulator/meshes/chain_link4.stl" scale="0.001 0.001 0.001"/>
+      </geometry>
+      <material name="grey"/>
+    </visual>
+    <collision>
+      <origin xyz="0 0 0" rpy="0 0 0"/>
+      <geometry>
+        <mesh filename="/home/kaito/ign_ws/src/open_manipulator_ign/models/openmanipulator/meshes/chain_link4.stl" scale="0.001 0.001 0.001"/>
       </geometry>
     </collision>
@@ -193,12 +193,12 @@
       <origin xyz="0 0 0" rpy="0 0 0"/>
       <geometry>
-        <mesh filename="package://open_manipulator_ign/models/openmanipulator/meshes/chain_link5.stl" scale="0.001 0.001 0.001"/>
-      </geometry>
-      <material name="grey"/>
-    </visual>
-    <collision>
-      <origin xyz="0 0 0" rpy="0 0 0"/>
-      <geometry>
-        <mesh filename="package://open_manipulator_ign/models/openmanipulator/meshes/chain_link5.stl" scale="0.001 0.001 0.001"/>
+        <mesh filename="/home/kaito/ign_ws/src/open_manipulator_ign/models/openmanipulator/meshes/chain_link5.stl" scale="0.001 0.001 0.001"/>
+      </geometry>
+      <material name="grey"/>
+    </visual>
+    <collision>
+      <origin xyz="0 0 0" rpy="0 0 0"/>
+      <geometry>
+        <mesh filename="/home/kaito/ign_ws/src/open_manipulator_ign/models/openmanipulator/meshes/chain_link5.stl" scale="0.001 0.001 0.001"/>
       </geometry>
     </collision>
@@ -223,5 +223,5 @@
       <origin xyz="0.0 0.0 0" rpy="0 0 0"/>
       <geometry>
-        <mesh filename="package://open_manipulator_ign/models/openmanipulator/meshes/chain_link_grip_l.stl" scale="0.001 0.001 0.001"/>
+        <mesh filename="/home/kaito/ign_ws/src/open_manipulator_ign/models/openmanipulator/meshes/chain_link_grip_l.stl" scale="0.001 0.001 0.001"/>
       </geometry>
       <material name="grey"/>
@@ -230,5 +230,5 @@
       <origin xyz="0.0 0.0 0" rpy="0 0 0"/>
       <geometry>
-        <mesh filename="package://open_manipulator_ign/models/openmanipulator/meshes/chain_link_grip_l.stl" scale="0.001 0.001 0.001"/>
+        <mesh filename="/home/kaito/ign_ws/src/open_manipulator_ign/models/openmanipulator/meshes/chain_link_grip_l.stl" scale="0.001 0.001 0.001"/>
       </geometry>
     </collision>
@@ -263,5 +263,5 @@
       <origin xyz="0.0 -0.0 0" rpy="0 0 0"/>
       <geometry>
-        <mesh filename="package://open_manipulator_ign/models/openmanipulator/meshes/chain_link_grip_r.stl" scale="0.001 0.001 0.001"/>
+        <mesh filename="/home/kaito/ign_ws/src/open_manipulator_ign/models/openmanipulator/meshes/chain_link_grip_r.stl" scale="0.001 0.001 0.001"/>
       </geometry>
       <material name="grey"/>
@@ -270,5 +270,5 @@
       <origin xyz="0.0 -0.0 0" rpy="0 0 0"/>
       <geometry>
-        <mesh filename="package://open_manipulator_ign/models/openmanipulator/meshes/chain_link_grip_r.stl" scale="0.001 0.001 0.001"/>
+        <mesh filename="/home/kaito/ign_ws/src/open_manipulator_ign/models/openmanipulator/meshes/chain_link_grip_r.stl" scale="0.001 0.001 0.001"/>
       </geometry>
     </collision>

Commit message: update urdf

File: worlds/openManipulator/open_manipulator.urdf (robot description, URDF)
Before this commit: robot open_manipulator, 9 links, 8 joints
Links:
- link gripper_link: geometry collision mesh filename=/home/kaito/catkin_ws/src/open_manipulator_ign/models/openm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 scale=0.001 0.001 0.001; visual mesh filename=/home/kaito/catkin_ws/src/open_manipulator_ign/models/openm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 scale=0.001 0.001 0.001
- link gripper_link_sub: geometry collision mesh filename=/home/kaito/catkin_ws/src/open_manipulator_ign/models/openm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 scale=0.001 0.001 0.001; visual mesh filename=/home/kaito/catkin_ws/src/open_manipulator_ign/models/openm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 scale=0.001 0.001 0.001
- link link1: geometry collision mesh filename=/home/kaito/catkin_ws/src/open_manipulator_ign/models/openm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 scale=0.001 0.001 0.001; visual mesh filename=/home/kaito/catkin_ws/src/open_manipulator_ign/models/openm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 scale=0.001 0.001 0.001
- link link2: geometry collision mesh filename=/home/kaito/catkin_ws/src/open_manipulator_ign/models/openm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 scale=0.001 0.001 0.001; visual mesh filename=/home/kaito/catkin_ws/src/open_manipulator_ign/models/openm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 scale=0.001 0.001 0.001
- link link3: geometry collision mesh filename=/home/kaito/catkin_ws/src/open_manipulator_ign/models/openm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 scale=0.001 0.001 0.001; visual mesh filename=/home/kaito/catkin_ws/src/open_manipulator_ign/models/openm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 scale=0.001 0.001 0.001
- link link4: geometry collision mesh filename=/home/kaito/catkin_ws/src/open_manipulator_ign/models/openm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 scale=0.001 0.001 0.001; visual mesh filename=/home/kaito/catkin_ws/src/open_manipulator_ign/models/openm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 scale=0.001 0.001 0.001
- link link5: geometry collision mesh filename=/home/kaito/catkin_ws/src/open_manipulator_ign/models/openm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 scale=0.001 0.001 0.001; visual mesh filename=/home/kaito/catkin_ws/src/open_manipulator_ign/models/openm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 scale=0.001 0.001 0.001
